File: kicad files/hackxpansion.kicad_pcb (KiCad board)
At the start: 2 copper layers, 32 x 25.5 mm, 12 parts, among them J2 Micro_SD_Card_Det1, SW1 SW_Push, SW2 SW_Push, SW3 SW_Push

Commit message: Add files via upload
Routing:
- net /P4: track 18.2 -> 27.5 mm
- net +3V3: track 44.5 -> 48.2 mm, vias 0 -> 1
- net Net-(J1-MD0): track 11.3 -> 7.92 mm
- net /P9: track 27.6 -> 30.4 mm, vias 2 -> 1
- net /BTN1: track 22.4 -> 19.9 mm, vias 1 -> 0
- net /P3: track 28.8 -> 31.0 mm, vias 1 -> 0
- net GND: vias 0 -> 7
- added copper zone on B.Cu, net GND
